File: substrate/Monea.sch (KiCad schematic (older format))
At the start: 5 parts

Commit message: :construction: WIP
Parts:
- added BZ1: Buzzer, symbol Device:Buzzer
- added D1: LED_RGBA, symbol Device:LED_RGBA
- gave numbers to parts that had none: 5
Connections:
- wire segments 43 -> 54
- no-connect marks 6 -> 35
Other:
- moved on the sheet: U1
Changed lines of the file:
@@
 $EndDescr
 $Comp
-L Connector_Generic:Conn_02x20_Odd_Even J?
+L Connector_Generic:Conn_02x20_Odd_Even J1
 U 1 1 61528489
 P 5000 3900
-F 0 "J?" H 5050 5017 50  0000 C CNN
+F 0 "J1" H 5050 5017 50  0000 C CNN
 F 1 "Conn_02x20_Odd_Even" H 5050 4926 50  0000 C CNN
 F 2 "" H 5000 3900 50  0001 C CNN
@@
 $EndComp
 $Comp
-L power:+5V #PWR?
+L power:+5V #PWR0101
 U 1 1 615297EB
 P 5600 2950
-F 0 "#PWR?" H 5600 2800 50  0001 C CNN
+F 0 "#PWR0101" H 5600 2800 50  0001 C CNN
 F 1 "+5V" H 5615 3123 50  0000 C CNN
 F 2 "" H 5600 2950 50  0001 C CNN
@@
 $EndComp
 $Comp
-L power:GND #PWR?
+L power:GND #PWR0102
 U 1 1 6152AB88
 P 5600 3250
-F 0 "#PWR?" H 5600 3000 50  0001 C CNN
+F 0 "#PWR0102" H 5600 3000 50  0001 C CNN
 F 1 "GND" H 5605 3077 50  0000 C CNN
 F 2 "" H 5600 3250 50  0001 C CNN
@@
 	5600 3200 5600 3250
 $Comp
-L Connector:Conn_01x06_Female J?
+L Connector:Conn_01x06_Female J2
 U 1 1 6152C049
 P 7300 3050
-F 0 "J?" H 7328 3026 50  0000 L CNN
+F 0 "J2" H 7328 3026 50  0000 L CNN
 F 1 "Conn_01x06_Female" H 7328 2935 50  0000 L CNN
 F 2 "" H 7300 3050 50  0001 C CNN
@@
 $EndComp
 $Comp
-L Connector:Conn_01x04_Female J?
+L Connector:Conn_01x04_Female J3
 U 1 1 6152DF10
 P 7300 3850
-F 0 "J?" H 7328 3826 50  0000 L CNN
+F 0 "J3" H 7328 3826 50  0000 L CNN
 F 1 "Conn_01x04_Female" H 7328 3735 50  0000 L CNN
 F 2 "" H 7300 3850 50  0001 C CNN
@@
 $EndComp
 $Comp
-L Connector:Conn_01x05_Female J?
+L Connector:Conn_01x05_Female J4
 U 1 1 6152E570
 P 7300 4450
-F 0 "J?" H 7328 4476 50  0000 L CNN
+F 0 "J4" H 7328 4476 50  0000 L CNN
 F 1 "Conn_01x05_Female" H 7328 4385 50  0000 L CNN
 F 2 "" H 7300 4450 50  0001 C CNN
@@
 $EndComp
 $Comp
-L power:+3.3V #PWR?
+L power:+3.3V #PWR0103
 U 1 1 61535927
 P 6800 2650
-F 0 "#PWR?" H 6800 2500 50  0001 C CNN
+F 0 "#PWR0103" H 6800 2500 50  0001 C CNN
 F 1 "+3.3V" H 6815 2823 50  0000 C CNN
 F 2 "" H 6800 2650 50  0001 C CNN
@@
 $EndComp
 $Comp
-L power:+3.3V #PWR?
+L power:+3.3V #PWR0104
 U 1 1 61535F16
 P 4500 2800
-F 0 "#PWR?" H 4500 2650 50  0001 C CNN
+F 0 "#PWR0104" H 4500 2650 50  0001 C CNN
 F 1 "+3.3V" H 4515 2973 50  0000 C CNN
 F 2 "" H 4500 2800 50  0001 C CNN
@@
 	6800 2850 7100 2850
 $Comp
-L power:GND #PWR?
+L power:GND #PWR0105
 U 1 1 61538D9A
 P 6800 4800
-F 0 "#PWR?" H 6800 4550 50  0001 C CNN
+F 0 "#PWR0105" H 6800 4550 50  0001 C CNN
 F 1 "GND" H 6805 4627 50  0000 C CNN
 F 2 "" H 6800 4800 50  0001 C CNN
@@
 	7100 2950 6800 2950
 Wire Wire Line
-	6800 2950 6800 3250
+	6800 2950 6800 3200
 Wire Wire Line
 	7100 3250 6800 3250
@@
 BME280
 $Comp
-L power:+5V #PWR?
+L power:+5V #PWR0106
 U 1 1 615BEF20
 P 7000 3700
-F 0 "#PWR?" H 7000 3550 50  0001 C CNN
+F 0 "#PWR0106" H 7000 3550 50  0001 C CNN
 F 1 "+5V" H 7015 3873 50  0000 C CNN
 F 2 "" H 7000 3700 50  0001 C CNN
@@
 Wire Wire Line
 	7100 3850 6800 3850
-Wire Wire Line
-	6800 3250 6800 3750
 Connection ~ 6800 3850
-Wire Wire Line
-	6800 3850 6800 4800
 NoConn ~ 7100 3950
 NoConn ~ 7100 4050
@@
 	5400 4450 7100 4450
 $Comp
-L LED:AE-WS2812B U?
+L LED:AE-WS2812B U1
 U 1 1 615CA3ED
-P 6050 3850
-F 0 "U?" H 6050 4182 50  0000 C CNN
-F 1 "AE-WS2812B" H 6050 4091 50  0000 C CNN
-F 2 "" H 6050 4050 50  0001 C CNN
-F 3 "" H 6050 4050 50  0001 C CNN
-	1    6050 3850
-	1    0    0    -1
-$EndComp
-Wire Wire Line
-	5600 3200 5750 3200
-Wire Wire Line
-	5750 3200 5750 3750
-Wire Wire Line
-	5750 3750 5850 3750
+P 8950 3950
+F 0 "U1" H 8950 4282 50  0000 C CNN
+F 1 "AE-WS2812B" H 8950 4191 50  0000 C CNN
+F 2 "" H 8950 4150 50  0001 C CNN
+F 3 "" H 8950 4150 50  0001 C CNN
+	1    8950 3950
+	1    0    0    -1
+$EndComp
+Wire Wire Line
+	8650 3300 8650 3850
+Wire Wire Line
+	8650 3850 8750 3850
 Connection ~ 5600 3200
 Wire Wire Line
-	6250 3750 6800 3750
-Connection ~ 6800 3750
-Wire Wire Line
-	6800 3750 6800 3850
-Wire Wire Line
-	6250 3950 7000 3950
-Wire Wire Line
-	7000 3950 7000 3750
-Connection ~ 7000 3750
-Wire Wire Line
-	7000 3950 7000 4100
-Wire Wire Line
-	7000 4100 5750 4100
-Wire Wire Line
-	5750 4100 5750 3950
-Wire Wire Line
-	5750 3950 5850 3950
-Connection ~ 7000 3950
+	9150 3850 9700 3850
+Wire Wire Line
+	9150 4050 9900 4050
+Wire Wire Line
+	9900 4200 8650 4200
+Wire Wire Line
+	8650 4200 8650 4050
+Wire Wire Line
+	8650 4050 8750 4050
+$Comp
+L Device:LED_RGBA D1
+U 1 1 6177CCDA
+P 6050 3900
+F 0 "D1" H 6050 4397 50  0000 C CNN
+F 1 "LED_RGBA" H 6050 4306 50  0000 C CNN
+F 2 "" H 6050 3850 50  0001 C CNN
+F 3 "~" H 6050 3850 50  0001 C CNN
+	1    6050 3900
+	1    0    0    -1
+$EndComp
+Wire Wire Line
+	6800 3250 6800 3850
+Wire Wire Line
+	5600 3200 6800 3200
+Connection ~ 6800 3200
+Wire Wire Line
+	6800 3200 6800 3250
+Wire Wire Line
+	6250 3900 6800 3900
+Wire Wire Line
+	6800 3850 6800 3900
+Connection ~ 6800 3900
+Wire Wire Line
+	6800 3900 6800 4800
+Wire Wire Line
+	5850 3700 5300 3700
+Wire Wire Line
+	5300 3800 5650 3800
+Wire Wire Line
+	5650 3800 5650 3900
+Wire Wire Line
+	5650 3900 5850 3900
+NoConn ~ 4800 3300
+NoConn ~ 4800 3400
+NoConn ~ 4800 3500
+NoConn ~ 4800 3600
+NoConn ~ 4800 3700
+NoConn ~ 4800 3800
+NoConn ~ 4800 3900
+NoConn ~ 4800 4000
+$Comp
+L Device:Buzzer BZ1
+U 1 1 61793657
+P 6050 4700
+F 0 "BZ1" H 6202 4729 50  0000 L CNN
+F 1 "Buzzer" H 6202 4638 50  0000 L CNN
+F 2 "" V 6025 4800 50  0001 C CNN
+F 3 "~" V 6025 4800 50  0001 C CNN
+	1    6050 4700
+	1    0    0    -1
+$EndComp
+Wire Wire Line
+	5950 4800 5450 4800
+Wire Wire Line
+	5450 4800 5450 4900
+Wire Wire Line
+	5450 4900 5300 4900
+$Comp
+L power:+5V #PWR0107
+U 1 1 61796161
+P 5750 4600
+F 0 "#PWR0107" H 5750 4450 50  0001 C CNN
+F 1 "+5V" H 5765 4773 50  0000 C CNN
+F 2 "" H 5750 4600 50  0001 C CNN
+F 3 "" H 5750 4600 50  0001 C CNN
+	1    5750 4600
+	1    0    0    -1
+$EndComp
+Wire Wire Line
+	5950 4600 5750 4600
+NoConn ~ 5300 4100
+NoConn ~ 5300 4200
+NoConn ~ 5300 4300
+NoConn ~ 5300 4400
+NoConn ~ 5300 4500
+NoConn ~ 5300 4600
+NoConn ~ 5300 4700
+NoConn ~ 5300 4800
+NoConn ~ 4800 4900
+NoConn ~ 4800 4800
+NoConn ~ 4800 4700
+NoConn ~ 4800 4600
+NoConn ~ 4800 4500
+NoConn ~ 4800 4400
+NoConn ~ 4800 4300
+NoConn ~ 4800 4200
+NoConn ~ 4800 4100
+NoConn ~ 5300 3100
+NoConn ~ 5300 3500
+NoConn ~ 5300 3600
+Wire Wire Line
+	5500 4100 5500 4000
+Wire Wire Line
+	5500 4000 5300 4000
+Wire Wire Line
+	5500 4100 5850 4100
+NoConn ~ 5300 3900
 $EndSCHEMATC

Commit message: :construction: WIP
Parts:
- removed U1: AE-WS2812B, symbol LED:AE-WS2812B
Connections:
- net labels removed: +3.3V, +5V, GND
- wire segments 54 -> 48
Changed lines of the file:
@@
 $EndComp
-$Comp
-L power:+5V #PWR0101
-U 1 1 615297EB
-P 5600 2950
-F 0 "#PWR0101" H 5600 2800 50  0001 C CNN
-F 1 "+5V" H 5615 3123 50  0000 C CNN
-F 2 "" H 5600 2950 50  0001 C CNN
-F 3 "" H 5600 2950 50  0001 C CNN
-	1    5600 2950
-	1    0    0    -1
-$EndComp
-$Comp
-L power:GND #PWR0102
-U 1 1 6152AB88
-P 5600 3250
-F 0 "#PWR0102" H 5600 3000 50  0001 C CNN
-F 1 "GND" H 5605 3077 50  0000 C CNN
-F 2 "" H 5600 3250 50  0001 C CNN
-F 3 "" H 5600 3250 50  0001 C CNN
-	1    5600 3250
-	1    0    0    -1
-$EndComp
-Wire Wire Line
-	5300 3000 5600 3000
-Wire Wire Line
-	5600 3000 5600 2950
-Wire Wire Line
-	5300 3200 5600 3200
-Wire Wire Line
-	5600 3200 5600 3250
 $Comp
 L Connector:Conn_01x06_Female J2
@@
 	1    0    0    -1
 $EndComp
-$Comp
-L power:+3.3V #PWR0103
-U 1 1 61535927
-P 6800 2650
-F 0 "#PWR0103" H 6800 2500 50  0001 C CNN
-F 1 "+3.3V" H 6815 2823 50  0000 C CNN
-F 2 "" H 6800 2650 50  0001 C CNN
-F 3 "" H 6800 2650 50  0001 C CNN
-	1    6800 2650
-	1    0    0    -1
-$EndComp
-$Comp
-L power:+3.3V #PWR0104
-U 1 1 61535F16
-P 4500 2800
-F 0 "#PWR0104" H 4500 2650 50  0001 C CNN
-F 1 "+3.3V" H 4515 2973 50  0000 C CNN
-F 2 "" H 4500 2800 50  0001 C CNN
-F 3 "" H 4500 2800 50  0001 C CNN
-	1    4500 2800
-	1    0    0    -1
-$EndComp
-Wire Wire Line
-	4500 2800 4500 3000
 Wire Wire Line
 	4500 3000 4800 3000
 Wire Wire Line
-	6800 2650 6800 2850
-Wire Wire Line
 	6800 2850 7100 2850
-$Comp
-L power:GND #PWR0105
-U 1 1 61538D9A
-P 6800 4800
-F 0 "#PWR0105" H 6800 4550 50  0001 C CNN
-F 1 "GND" H 6805 4627 50  0000 C CNN
-F 2 "" H 6800 4800 50  0001 C CNN
-F 3 "" H 6800 4800 50  0001 C CNN
-	1    6800 4800
-	1    0    0    -1
-$EndComp
 Wire Wire Line
 	7100 2950 6800 2950
@@
 Text Notes 7150 2750 0    50   ~ 0
 BME280
-$Comp
-L power:+5V #PWR0106
-U 1 1 615BEF20
-P 7000 3700
-F 0 "#PWR0106" H 7000 3550 50  0001 C CNN
-F 1 "+5V" H 7015 3873 50  0000 C CNN
-F 2 "" H 7000 3700 50  0001 C CNN
-F 3 "" H 7000 3700 50  0001 C CNN
-	1    7000 3700
-	1    0    0    -1
-$EndComp
-Wire Wire Line
-	7000 3700 7000 3750
 Wire Wire Line
 	7000 3750 7100 3750
@@
 	5400 4450 7100 4450
 $Comp
-L LED:AE-WS2812B U1
-U 1 1 615CA3ED
-P 8950 3950
-F 0 "U1" H 8950 4282 50  0000 C CNN
-F 1 "AE-WS2812B" H 8950 4191 50  0000 C CNN
-F 2 "" H 8950 4150 50  0001 C CNN
-F 3 "" H 8950 4150 50  0001 C CNN
-	1    8950 3950
-	1    0    0    -1
-$EndComp
-Wire Wire Line
-	8650 3300 8650 3850
-Wire Wire Line
-	8650 3850 8750 3850
-Connection ~ 5600 3200
-Wire Wire Line
-	9150 3850 9700 3850
-Wire Wire Line
-	9150 4050 9900 4050
-Wire Wire Line
-	9900 4200 8650 4200
-Wire Wire Line
-	8650 4200 8650 4050
-Wire Wire Line
-	8650 4050 8750 4050
-$Comp
 L Device:LED_RGBA D1
 U 1 1 6177CCDA
@@
 Wire Wire Line
 	6800 3250 6800 3850
-Wire Wire Line
-	5600 3200 6800 3200
 Connection ~ 6800 3200
 Wire Wire Line
@@
 Wire Wire Line
 	6800 3850 6800 3900
-Connection ~ 6800 3900
-Wire Wire Line
-	6800 3900 6800 4800
 Wire Wire Line
 	5850 3700 5300 3700
@@
 Wire Wire Line
 	5450 4900 5300 4900
-$Comp
-L power:+5V #PWR0107
-U 1 1 61796161
-P 5750 4600
-F 0 "#PWR0107" H 5750 4450 50  0001 C CNN
-F 1 "+5V" H 5765 4773 50  0000 C CNN
-F 2 "" H 5750 4600 50  0001 C CNN
-F 3 "" H 5750 4600 50  0001 C CNN
-	1    5750 4600
-	1    0    0    -1
-$EndComp
 Wire Wire Line
-	5950 4600 5750 4600
+	5950 4600 5900 4600
 NoConn ~ 5300 4100
 NoConn ~ 5300 4200
@@
 	5500 4100 5850 4100
 NoConn ~ 5300 3900
+Wire Wire Line
+	4500 3000 4500 2500
+Wire Wire Line
+	4500 2500 6800 2500
+Wire Wire Line
+	6800 2500 6800 2850
+Wire Wire Line
+	6500 3000 6500 3750
+Wire Wire Line
+	6500 3750 7000 3750
+Connection ~ 7000 3750
+Wire Wire Line
+	5900 4600 5900 4300
+Wire Wire Line
+	5900 4300 7000 4300
+Wire Wire Line
+	7000 4300 7000 3750
+Wire Wire Line
+	5300 3200 6800 3200
+Wire Wire Line
+	5300 3000 6500 3000
 $EndSCHEMATC

Commit message: :construction: WIP
Connections:
- net +3V3: now reaches J1.1 (Pin_1), J2.1 (Pin_1)
- net RX: now reaches J1.10 (Pin_10), J4.3 (Pin_3)
- net R: now reaches J1.12 (Pin_12)
- net R: now also D1.1 (RK)
- net G: now reaches J1.16 (Pin_16)
- net G: now also D1.2 (GK); no longer D1.1 (RK)
- net B: now reaches J1.18 (Pin_18)
- net B: now also D1.3 (BK); no longer D1.2 (GK)
- net +5V: now reaches J1.2 (Pin_2), J3.1 (Pin_1)
- net +5V: no longer BZ1.1 (-)
- net at J1.22 (Pin_22): no longer D1.3 (BK)
- net SDA: now reaches J1.3 (Pin_3), J2.4 (Pin_4)
- net at J1.40 (Pin_40): no longer BZ1.2 (+)
- net SCL: now reaches J1.5 (Pin_5), J2.6 (Pin_6)
- net GND: now reaches D1.4 (A), J1.6 (Pin_6), J2.2 (Pin_2), J2.5 (Pin_5), J3.2 (Pin_2)
- net GND: now also BZ1.2 (+)
- net BZ: now reaches J1.7 (Pin_7)
- net BZ: now also BZ1.1 (-)
- net TX: now reaches J1.8 (Pin_8), J4.2 (Pin_2)
- no-connect marks 35 -> 34
Other:
- note added: "Buzzer"
- note added: "Color LED"
- note added: "MH-Z19C"
- note added: "Raspberry Pi Zero"
- note removed: "RX"
- moved on the sheet: BZ1, D1, J2, J3, J4

Commit message: :construction: WIP
Parts:
- removed D1: LED_RGBA, symbol Device:LED_RGBA
- added D1: LED_GBCR, LED_THT:LED_D5.0mm-4_RGB, symbol Device:LED_GBCR
- added R1: R, Resistor_THT:R_Axial_DIN0204_L3.6mm_D1.6mm_P5.08mm_Horizontal, symbol Device:R
- BZ1: footprint (none) -> Buzzer_Beeper:Buzzer_12x9.5RM7.6
- J1: footprint (none) -> Connector_PinSocket_2.54mm:PinSocket_2x40_P2.54mm_Vertical
- J2: footprint (none) -> Connector_PinSocket_2.54mm:PinSocket_1x06_P2.54mm_Vertical
- J3: footprint (none) -> Connector_PinSocket_2.54mm:PinSocket_1x04_P2.54mm_Vertical
- J4: footprint (none) -> Connector_PinSocket_2.54mm:PinSocket_1x05_P2.54mm_Vertical
Connections:
- net B: now also J1.16 (Pin_16), D1.2 (BA); no longer J1.18 (Pin_18)
- net G: now also J1.13 (Pin_13), D1.1 (GA); no longer J1.16 (Pin_16)
- net GND: now also D1.3 (K)
- net R: now also D1.4 (RA), R1.2; no longer J1.12 (Pin_12)
- net at J1.11 (Pin_11): now also R1.1
- no-connect marks 34 -> 35
Changed lines of the file:
@@
 F 0 "J1" H 5050 5000 50  0000 C CNN
 F 1 "Conn_02x20_Odd_Even" H 5100 4900 50  0000 C CNN
-F 2 "" H 5000 3900 50  0001 C CNN
+F 2 "Connector_PinSocket_2.54mm:PinSocket_2x40_P2.54mm_Vertical" H 5000 3900 50  0001 C CNN
 F 3 "~" H 5000 3900 50  0001 C CNN
 	1    5000 3900
@@
 F 0 "J2" H 6250 3550 50  0000 L CNN
 F 1 "Conn_01x06_Female" H 5750 3450 50  0000 L CNN
-F 2 "" H 6400 4150 50  0001 C CNN
+F 2 "Connector_PinSocket_2.54mm:PinSocket_1x06_P2.54mm_Vertical" H 6400 4150 50  0001 C CNN
 F 3 "~" H 6400 4150 50  0001 C CNN
 	1    6400 4150
@@
 F 0 "J3" H 6900 3600 50  0000 L CNN
 F 1 "Conn_01x04_Female" H 6600 3500 50  0000 L CNN
-F 2 "" H 7000 3900 50  0001 C CNN
+F 2 "Connector_PinSocket_2.54mm:PinSocket_1x04_P2.54mm_Vertical" H 7000 3900 50  0001 C CNN
 F 3 "~" H 7000 3900 50  0001 C CNN
 	1    7000 3900
@@
 F 0 "J4" H 6850 4400 50  0000 L CNN
 F 1 "Conn_01x05_Female" H 6600 4300 50  0000 L CNN
-F 2 "" H 6950 4650 50  0001 C CNN
+F 2 "Connector_PinSocket_2.54mm:PinSocket_1x05_P2.54mm_Vertical" H 6950 4650 50  0001 C CNN
 F 3 "~" H 6950 4650 50  0001 C CNN
 	1    6950 4650
@@
 NoConn ~ 6750 4750
 NoConn ~ 6750 4850
-$Comp
-L Device:LED_RGBA D1
-U 1 1 6177CCDA
-P 6950 3150
-F 0 "D1" H 6950 3647 50  0000 C CNN
-F 1 "LED_RGBA" H 6950 3556 50  0000 C CNN
-F 2 "" H 6950 3100 50  0001 C CNN
-F 3 "~" H 6950 3100 50  0001 C CNN
-	1    6950 3150
-	1    0    0    -1
-$EndComp
 NoConn ~ 4800 3400
-NoConn ~ 4800 3500
-NoConn ~ 4800 3600
 NoConn ~ 4800 3700
 NoConn ~ 4800 3800
@@
 F 0 "BZ1" H 6150 2850 50  0000 L CNN
 F 1 "Buzzer" H 6100 2750 50  0000 L CNN
-F 2 "" V 6125 3150 50  0001 C CNN
+F 2 "Buzzer_Beeper:Buzzer_12x9.5RM7.6" V 6125 3150 50  0001 C CNN
 F 3 "~" V 6125 3150 50  0001 C CNN
 	1    6150 3050
@@
 NoConn ~ 5300 4700
 NoConn ~ 5300 4800
-NoConn ~ 4800 4900
 NoConn ~ 4800 4800
 NoConn ~ 4800 4700
@@
 NoConn ~ 4800 4100
 NoConn ~ 5300 3100
-NoConn ~ 5300 3600
 NoConn ~ 5300 3900
 Text GLabel 4800 3100 0    50   Input ~ 0
@@
 L power:GND #PWR0103
 U 1 1 61A08987
-P 5550 3300
-F 0 "#PWR0103" H 5550 3050 50  0001 C CNN
-F 1 "GND" H 5555 3127 50  0000 C CNN
-F 2 "" H 5550 3300 50  0001 C CNN
-F 3 "" H 5550 3300 50  0001 C CNN
-	1    5550 3300
-	1    0    0    -1
-$EndComp
-Wire Wire Line
-	5300 3200 5550 3200
-Wire Wire Line
-	5550 3200 5550 3300
+P 5550 3250
+F 0 "#PWR0103" H 5550 3000 50  0001 C CNN
+F 1 "GND" H 5555 3077 50  0000 C CNN
+F 2 "" H 5550 3250 50  0001 C CNN
+F 3 "" H 5550 3250 50  0001 C CNN
+	1    5550 3250
+	1    0    0    -1
+$EndComp
 $Comp
 L power:GND #PWR0104
@@
 Text GLabel 6750 2950 0    50   Input ~ 0
 R
-Text GLabel 5300 3500 2    50   Input ~ 0
-R
-Text GLabel 5300 3700 2    50   Input ~ 0
-G
-Text GLabel 5300 3800 2    50   Input ~ 0
-B
 NoConn ~ 5300 4000
 Text GLabel 6750 3150 0    50   Input ~ 0
@@
 Wire Wire Line
 	4600 3000 4800 3000
-Text Notes 4500 5150 0    50   ~ 0
+Text Notes 5000 5150 0    50   ~ 0
 Raspberry Pi Zero
 Text Notes 6250 3550 0    50   ~ 0
@@
 Wire Wire Line
 	6000 3300 6000 3150
+$Comp
+L Device:LED_GBCR D1
+U 1 1 61AEEBA7
+P 6950 3150
+F 0 "D1" H 6950 3647 50  0000 C CNN
+F 1 "LED_GBCR" H 6950 3556 50  0000 C CNN
+F 2 "LED_THT:LED_D5.0mm-4_RGB" H 6950 3100 50  0001 C CNN
+F 3 "~" H 6950 3100 50  0001 C CNN
+	1    6950 3150
+	-1   0    0    -1
+$EndComp
+Text GLabel 4600 4150 3    50   Input ~ 0
+R
+Text GLabel 4800 3600 0    50   Input ~ 0
+G
+Text GLabel 5300 3700 2    50   Input ~ 0
+B
+NoConn ~ 5300 3800
+NoConn ~ 5300 4900
+NoConn ~ 5300 3500
+NoConn ~ 5300 3600
+Wire Wire Line
+	4800 3500 4600 3500
+Wire Wire Line
+	4600 3500 4600 3700
+$Comp
+L Device:R R1
+U 1 1 61B088E8
+P 4600 3850
+F 0 "R1" H 4670 3896 50  0000 L CNN
+F 1 "R" H 4670 3805 50  0000 L CNN
+F 2 "Resistor_THT:R_Axial_DIN0204_L3.6mm_D1.6mm_P5.08mm_Horizontal" V 4530 3850 50  0001 C CNN
+F 3 "~" H 4600 3850 50  0001 C CNN
+	1    4600 3850
+	1    0    0    -1
+$EndComp
+Wire Wire Line
+	4600 4000 4600 4150
+Wire Wire Line
+	5550 3200 5550 3250
+Wire Wire Line
+	5300 3200 5550 3200
+NoConn ~ 4800 4900
 $EndSCHEMATC
